File: RMF_Driver/RMF_Driver.kicad_sch (KiCad schematic)
At the start: 1 part

Commit message: updated to rev B
Parts:
- removed LED?: (no value), symbol RMF_Bi-Color_LED:VLMKG3400-GS18
Other:
- added sheet Clock and Frequency Generator (Clock_and_Frequency_Generator.kicad_sch)
- added sheet Logic (Logic.kicad_sch)
- added sheet Mosfet Coil Driver (Mosfet_Coil_Driver.kicad_sch)
- added sheet Power In Terminals | Temp Sensor | Power Supply (PowerInConnTempSensor.kicad_sch)
- title: (none) -> RMF Driver
